File: Bal_St_4_1_Mux.sch (KiCad schematic (older format))
At the start: 2 parts

Commit message: Rename power flags for consistency
Connections:
- net labels added: VA+, VA-
- net labels removed: +VA, -VA
Changed lines of the file:
@@
 $Descr A4 11693 8268
 encoding utf-8
-Sheet 12 13
+Sheet 8 13
 Title "Monitor Control"
 Date ""
@@
 $EndComp
 Text GLabel 6050 4550 1    50   Input ~ 0
-+VA
+VA+
 Text GLabel 6050 2700 1    50   Input ~ 0
-+VA
+VA+
 Text GLabel 6050 4150 3    50   Input ~ 0
--VA
+VA-
 Text GLabel 6050 6000 3    50   Input ~ 0
--VA
+VA-
 Wire Wire Line
 	6800 3650 7900 3650
