File: Headphone_out.sch (KiCad schematic (older format))
At the start: 16 parts

Commit message: Rename power flags for consistency
Connections:
- net labels added: VA+, VA-
- net labels removed: +VA, -VA
Changed lines of the file:
@@
 R+
 Text GLabel 5200 1500 1    50   Input ~ 0
-+VA
+VA+
 Text GLabel 5200 4650 3    50   Input ~ 0
--VA
+VA-
 $Comp
 L Device:C C?
